File: arduinoNano/arduinoNano.kicad_pcb (KiCad board)
At the start: 4 copper layers, 45 x 19 mm, 35 parts, among them J1 USB_B_Mini, J2 Conn_01x15_Pin, J3 ICSP, J4 Conn_01x15_Pin, J5 ICSP, SW1 SW_Push, U1 LM1117MP-5.0, U2 ATmega328P-M, U3 FT232RL, Y1 16MHz

Commit message: pcb design in process
Parts:
- moved J3 91.1 mm to (139.8, 61.9), turned to 180 degrees
- moved J5 89.8 mm to (143.1, 61.9), turned to 180 degrees
- moved SW1 86.9 mm to (135.6, 59.4), turned to 90 degrees
- moved C4 72.9 mm to (112.9, 64.1)
- moved C6 6.25 mm to (125.3, 63.0)
- moved U1 4.20 mm to (131.2, 61.0)
- moved C5 4.20 mm to (136.5, 61.4)
- moved D1 1.52 mm to (112.9, 61.8), turned to 0 degrees
- moved C2 0.41 mm to (125.0, 56.5)
Routing:
- net (no net): vias 0 -> 2

Commit message: Done designing, next will be wiring
Parts:
- D2, D4, D5, R5, R6, R7, TP1, TP2: moved to B.Cu
- moved R1 102.8 mm to (133.8, 54.7)
- moved R3 98.0 mm to (127.6, 63.4), turned to -90 degrees
- moved R2 97.4 mm to (125.9, 63.4), turned to -90 degrees
- moved D5 92.5 mm to (122.9, 59.4), turned to -90 degrees
- moved D4 90.7 mm to (120.8, 59.4), turned to -90 degrees
- moved R7 88.1 mm to (122.4, 55.7), turned to 90 degrees
- moved R6 87.0 mm to (120.7, 55.9), turned to 90 degrees
- moved D3 82.6 mm to (113.8, 56.2), turned to 90 degrees
- moved TP2 60.0 mm to (105.0, 54.8), turned to 180 degrees
- moved TP1 57.4 mm to (102.5, 55.0), turned to 180 degrees
- moved D2 43.7 mm to (135.5, 55.4), turned to 180 degrees
- moved R5 41.9 mm to (131.9, 55.4), turned to 180 degrees
- moved D1 17.8 mm to (130.5, 59.2)
- moved R4 4.92 mm to (111.5, 62.2), turned to 180 degrees
- moved C4 4.58 mm to (112.0, 59.6), turned to 180 degrees
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Routing:
- net /XTAL2: vias 0 -> 1
- net /XTAL1: vias 0 -> 1
- net (no net): vias 2 -> 0
